File: PCB/macropad.kicad_pcb (KiCad board)
At the start: 2 copper layers, 69.1 x 88.1 mm, 33 parts, among them SW1 SW_Push, SW10 SW_Push, SW11 SW_Push, SW12 SW_Push, SW13 SW_Push, SW14 SW_Push, SW15 SW_Push, SW16 SW_Push, SW2 SW_Push, SW3 SW_Push, SW4 SW_Push, SW5 SW_Push, SW6 SW_Push, SW7 SW_Push, SW8 SW_Push, SW9 SW_Push, U2 MOUDLE-SEEEDUINO-XIAO

Commit message: Start of case
Parts:
- added ?: , , F.Cu at (119.1, 137.3)
- added ?: , , F.Cu at (119.1, 51.6)
- added ?: , , F.Cu at (192.1, 137.3)
- added REF**: MountingHole_3.2mm_M3_Pad, MountingHole:MountingHole_3.2mm_M3_Pad, F.Cu at (192.1, 51.6)
Other:
- board size 69.1 x 88.1 mm -> 81.1 x 93.4 mm
Changed lines of the file:
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@@
     )
+  )
+  (footprint "" (layer "F.Cu")
+    (at 119.0625 137.31875)
+    (fp_text reference "" (at 0 0) (layer "F.SilkS")
+        (effects (font (size 1.27 1.27) (thickness 0.15)))
+    )
+    (fp_text value "" (at 0 0) (layer "F.SilkS")
+        (effects (font (size 1.27 1.27) (thickness 0.15)))
+    )
+    (pad "1" thru_hole circle (at 0 0) (size 6.4 6.4) (drill 3.2) (layers "*.Cu" "*.Mask")
+      (net 26 "GND"))
   )
   (footprint "key:SW_Kailh_Choc_V2_THT" (layer "F.Cu")
@@
     )
   )
+  (footprint "MountingHole:MountingHole_3.2mm_M3_Pad" (layer "F.Cu")
+    (at 192.0875 51.59375)
+    (descr "Mounting Hole 3.2mm, M3")
+    (tags "mounting hole 3.2mm m3")
+    (attr exclude_from_pos_files exclude_from_bom)
+    (fp_text reference "REF**" (at 0 -4.2) (layer "F.SilkS") hide
+        (effects (font (size 1 1) (thickness 0.15)))
+    )
+    (fp_text value "MountingHole_3.2mm_M3_Pad" (at 0 4.2) (layer "F.Fab") hide
+        (effects (font (size 1 1) (thickness 0.15)))
+    )
+    (fp_text user "${REFERENCE}" (at 0 0) (layer "F.Fab")
+        (effects (font (size 1 1) (thickness 0.15)))
+    )
+    (fp_circle (center 0 0) (end 3.2 0)
+      (stroke (width 0.15) (type solid)) (fill none) (layer "Cmts.User"))
+    (fp_circle (center 0 0) (end 3.45 0)
+      (stroke (width 0.05) (type solid)) (fill none) (layer "F.CrtYd"))
+    (pad "1" thru_hole circle (at 0 0) (size 6.4 6.4) (drill 3.2) (layers "*.Cu" "*.Mask")
+      (net 26 "GND"))
+  )
   (footprint "key:SW_Kailh_Choc_V2_THT" (layer "F.Cu")
     (at 180.38445 78.72645)
@@
     )
   )
+  (footprint "" (layer "F.Cu")
+    (at 119.0625 51.59375)
+    (fp_text reference "" (at 0 0) (layer "F.SilkS")
+        (effects (font (size 1.27 1.27) (thickness 0.15)))
+    )
+    (fp_text value "" (at 0 0) (layer "F.SilkS")
+        (effects (font (size 1.27 1.27) (thickness 0.15)))
+    )
+    (pad "1" thru_hole circle (at 0 0) (size 6.4 6.4) (drill 3.2) (layers "*.Cu" "*.Mask")
+      (net 26 "GND"))
+  )
+  (footprint "" (layer "F.Cu")
+    (at 192.0875 137.31875)
+    (fp_text reference "" (at 0 0) (layer "F.SilkS")
+        (effects (font (size 1.27 1.27) (thickness 0.15)))
+    )
+    (fp_text value "" (at 0 0) (layer "F.SilkS")
+        (effects (font (size 1.27 1.27) (thickness 0.15)))
+    )
+    (pad "1" thru_hole circle (at 0 0) (size 6.4 6.4) (drill 3.2) (layers "*.Cu" "*.Mask")
+      (net 26 "GND"))
+  )
   (footprint "Diode_THT:D_DO-35_SOD27_P7.62mm_Horizontal" (layer "B.Cu")
     (at 169.27195 60.3377 -90)
@@
     )
   )
-  (gr_line (start 186.73445 52.87645) (end 124.0282 52.87645)
+  (gr_line (start 193.017421 47.625) (end 118.26875 47.625)
     (stroke (width 0.05) (type default)) (layer "Edge.Cuts"))
-  (gr_arc (start 189.90945 137.8077) (mid 188.979514 140.052764) (end 186.73445 140.9827)
+  (gr_arc (start 196.192421 137.8077) (mid 195.262488 140.052782) (end 193.017421 140.9827)
     (stroke (width 0.05) (type default)) (layer "Edge.Cuts"))
-  (gr_line (start 120.8532 56.05145) (end 120.8532 137.8077)
+  (gr_line (start 115.09375 50.8) (end 115.09375 137.8077)
     (stroke (width 0.05) (type default)) (layer "Edge.Cuts"))
-  (gr_arc (start 186.73445 52.87645) (mid 188.979532 53.806383) (end 189.90945 56.05145)
+  (gr_arc (start 193.017421 47.625) (mid 195.2625 48.554921) (end 196.192421 50.8)
     (stroke (width 0.05) (type default)) (layer "Edge.Cuts"))
-  (gr_line (start 189.90945 137.8077) (end 189.90945 56.05145)
+  (gr_line (start 196.192421 137.8077) (end 196.192421 50.8)
     (stroke (width 0.05) (type default)) (layer "Edge.Cuts"))
-  (gr_arc (start 124.0282 140.9827) (mid 121.783168 140.052746) (end 120.8532 137.8077)
+  (gr_arc (start 118.26875 140.9827) (mid 116.023715 140.052735) (end 115.09375 137.8077)
     (stroke (width 0.05) (type default)) (layer "Edge.Cuts"))
-  (gr_line (start 124.0282 140.9827) (end 186.73445 140.9827)
+  (gr_line (start 119.720046 140.9827) (end 193.017421 140.9827)
     (stroke (width 0.05) (type default)) (layer "Edge.Cuts"))
-  (gr_arc (start 120.8532 56.05145) (mid 121.783136 53.806386) (end 124.0282 52.87645)
+  (gr_arc (start 115.09375 50.8) (mid 116.023704 48.554968) (end 118.26875 47.625)
     (stroke (width 0.05) (type default)) (layer "Edge.Cuts"))
   (segment (start 129.12725 65.8749) (end 127.01905 67.9831) (width 0.4) (layer "F.Cu") (net 1))
@@
     (polygon
       (pts
-        (xy 190.0428 140.9192)
-        (xy 189.992 52.7304)
-        (xy 120.5484 52.7812)
-        (xy 120.8024 141.0208)
+        (xy 196.85 141.2875)
+        (xy 196.85 47.625)
+        (xy 114.3 47.625)
+        (xy 114.3 141.2875)
       )
     )

Commit message: Fix stuff
Parts:
- ?: moved to B.Cu
- moved ? 0.79 mm to (192.1, 136.5)
- moved ? 0.79 mm to (119.1, 136.5), turned to 180 degrees
Other:
- outline, holes or cut-outs redrawn
Changed lines of the file:
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@@
     )
-  )
-  (footprint "" (layer "F.Cu")
-    (at 119.0625 137.31875)
-    (fp_text reference "" (at 0 0) (layer "F.SilkS")
-        (effects (font (size 1.27 1.27) (thickness 0.15)))
-    )
-    (fp_text value "" (at 0 0) (layer "F.SilkS")
-        (effects (font (size 1.27 1.27) (thickness 0.15)))
-    )
-    (pad "1" thru_hole circle (at 0 0) (size 6.4 6.4) (drill 3.2) (layers "*.Cu" "*.Mask")
-      (net 26 "GND"))
   )
   (footprint "key:SW_Kailh_Choc_V2_THT" (layer "F.Cu")
@@
   )
   (footprint "" (layer "F.Cu")
-    (at 192.0875 137.31875)
+    (at 192.0875 136.525)
     (fp_text reference "" (at 0 0) (layer "F.SilkS")
         (effects (font (size 1.27 1.27) (thickness 0.15)))
@@
       (rotate (xyz 0 0 0))
     )
+  )
+  (footprint "" (layer "B.Cu")
+    (at 119.0625 136.525 180)
+    (fp_text reference "" (at 0 0) (layer "B.SilkS")
+        (effects (font (size 1.27 1.27) (thickness 0.15)) (justify mirror))
+    )
+    (fp_text value "" (at 0 0) (layer "B.SilkS")
+        (effects (font (size 1.27 1.27) (thickness 0.15)) (justify mirror))
+    )
+    (pad "1" thru_hole circle (at 0 0 180) (size 6.4 6.4) (drill 3.2) (layers "*.Cu" "*.Mask")
+      (net 26 "GND"))
   )
   (footprint "seed:XIAO-SAMD21-RP2040-14P-2.54-21X17.8MM (Seeeduino XIAO)" (layer "B.Cu")
@@
   (gr_arc (start 118.26875 140.9827) (mid 116.023715 140.052735) (end 115.09375 137.8077)
     (stroke (width 0.05) (type default)) (layer "Edge.Cuts"))
-  (gr_line (start 119.720046 140.9827) (end 193.017421 140.9827)
+  (gr_line (start 118.26875 140.9827) (end 193.017421 140.9827)
     (stroke (width 0.05) (type default)) (layer "Edge.Cuts"))
   (gr_arc (start 115.09375 50.8) (mid 116.023704 48.554968) (end 118.26875 47.625)

Commit message: Silkscreen
Parts:
- added Gura!: LOGO, LOGO, F.Cu at (136.5, 130.2)
Other:
- board text added: "By Cyao"
- board text added: "UwU"

Commit message: LCD!
Parts:
- added Brd1: SSD1306, screen:128x64OLED, F.Cu at (163.6, 63.1)
- added H1: MountingHole_Pad, Connector_Wire:SolderWire-0.1sqmm_1x01_D0.4mm_OD1mm, F.Cu at (184.2, 58.7)
- moved ? 122.2 mm to (200.1, 143.1), turned to 180 degrees
- moved ? 115.6 mm to (200.1, 54.2), turned to 0 degrees
- moved REF** 113.6 mm to (124.7, 143.1), turned to 180 degrees
- moved ? 106.4 mm to (124.7, 54.2), turned to 180 degrees
- moved U2 75.7 mm to (184.3, 60.5), turned to 180 degrees
- moved Gura! 66.0 mm to (140.5, 64.3)
- moved D1 26.1 mm to (143.0, 85.4)
- moved D10 26.1 mm to (193.0, 85.4)
- moved D11 26.1 mm to (193.0, 102.1)
- moved D12 26.1 mm to (193.0, 118.8)
- moved D2 26.1 mm to (159.7, 85.4)
- moved D4 26.1 mm to (143.0, 102.1)
- moved D5 26.1 mm to (159.7, 102.1)
- moved D7 26.1 mm to (143.0, 118.8)
- moved D8 26.1 mm to (159.7, 118.8)
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Connections:
- U2 pad 1: unconnected-(U2-PA02_A0_D0-Pad1) -> Net-(U2-PA02_A0_D0)
- U2 pad 10: COL2 -> COL1
- U2 pad 11: COL3 -> COL0
- U2 pad 2: unconnected-(U2-PA4_A1_D1-Pad2) -> ROW0
- U2 pad 3: unconnected-(U2-PA10_A2_D2-Pad3) -> ROW3
- U2 pad 4: COL0 -> ROW2
- U2 pad 5: COL1 -> Net-(Brd1-SDA)
- U2 pad 6: ROW0 -> Net-(Brd1-SCL)
- U2 pad 8: ROW2 -> COL3
- U2 pad 9: ROW3 -> COL2
Routing:
- net ROW0: track 142.5 -> 86.8 mm, vias 1 -> 0
- net ROW3: track 93.4 -> 138.8 mm
- net COL0: track 78.0 -> 115.9 mm, vias 0 -> 1
- net COL1: track 66.1 -> 101.7 mm, vias 0 -> 1
- net Net-(Brd1-SCL): track 0.00 -> 34.6 mm, vias 0 -> 1
- net Net-(Brd1-SDA): track 0.00 -> 31.2 mm, vias 0 -> 1
- net ROW2: track 91.1 -> 118.1 mm, vias 1 -> 0
- net COL2: track 66.4 -> 83.3 mm, vias 0 -> 1
- net +5V: track 0.00 -> 15.9 mm
- net ROW1: track 107.3 -> 92.2 mm, vias 1 -> 0
- net Net-(U2-PA02_A0_D0): track 0.00 -> 12.0 mm
- net COL3: track 73.3 -> 75.6 mm, vias 0 -> 1
- net GND: vias 14 -> 50
Other:
- board size 81.1 x 93.4 mm -> 83.5 x 97.3 mm
- board text removed: "UwU"
